Commit message: Update mixed ROS1/ROS2 platform, PX4 launch flow, and Phase 1 artifacts

File: catkin_ws_src/wamv_description/urdf/wamv_base.urdf.xacro (robot description, xacro)
@@ -94,9 +94,9 @@
       </geometry>
     </visual>
-    <!-- 添加二维码模型 -->
+    <!-- AprilTag marker mounted on the deck landing target -->
     <visual name="marker_visual">
-      <origin xyz="-0.5 0 1.3" rpy="0 1.57 0" /> <!-- 调整二维码的位置 -->
+      <origin xyz="-0.5 0 1.3" rpy="0 1.57 0" />
       <geometry>
-        <mesh filename="package://wamv_description/models/marker0/meshes/Marker0.dae" scale="2 2 2" />
+        <mesh filename="package://wamv_description/models/tag/meshes/tag.dae" scale="4 4 4" />
       </geometry>
     </visual>
